File: track-voltage.kicad_pcb (KiCad board)
At the start: 2 copper layers, 12 parts, among them J3 Screw_Terminal_01x02

Commit message: Add PCB.
Parts:
- added J1: PAD, TestPoint:TestPoint_Pad_1.0x1.0mm, F.Cu at (192.0, 113.0)
- added J2: MPB1, track-voltage:MPB1, F.Cu at (192.4, 91.4)
- added J4: PAD, TestPoint:TestPoint_Pad_1.0x1.0mm, F.Cu at (173.2, 113.0)
- added J5: MPB1, track-voltage:MPB1, F.Cu at (172.7, 91.4)
- D3: value D_Bridge_+-AA -> S250; footprint Diode_SMD:Diode_Bridge_Diotec_SO-DIL-Slim -> track-voltage:S250
- moved TP1 50.5 mm to (190.0, 97.0)
- moved D1 38.9 mm to (184.7, 109.7), turned to 180 degrees
- moved D3 38.0 mm to (182.4, 102.4), turned to 270 degrees
- moved D4 35.9 mm to (180.1, 89.4)
- moved J3 34.7 mm to (183.6, 82.5), turned to 270 degrees
- moved R2 34.3 mm to (180.1, 109.7)
- moved R3 30.0 mm to (184.6, 89.4), turned to 180 degrees
- moved R1 29.8 mm to (184.6, 113.0), turned to 180 degrees
- moved D2 27.3 mm to (180.1, 113.0)
- moved TP2 23.3 mm to (174.8, 97.3)
- moved R4 21.8 mm to (182.4, 92.2), turned to 180 degrees
- moved C1 20.2 mm to (182.4, 95.5), turned to 180 degrees
Routing:
- net Net-(D4-Pad2): track 0.00 -> 2.54 mm
- net Net-(D2-Pad2): track 0.00 -> 2.54 mm
- net Net-(D1-Pad2): track 0.00 -> 2.54 mm
- net VCC: vias 0 -> 4
- net GND: vias 0 -> 4
- net /K: vias 0 -> 10
- net /J: vias 0 -> 10
- added copper zone on B.Cu, net /J
- added copper zone on F.Cu, net /J
- added copper zone on B.Cu, net /K
- added copper zone on F.Cu, net /K
- added copper zone on B.Cu, net GND
- added copper zone on F.Cu, net GND
- added copper zone on B.Cu, net VCC
- added copper zone on F.Cu, net VCC
Other:
- board outline added: 25 x 40 mm
- board text added: "+"
- board text added: "-"
- board text added: "Track voltage rectifier"
- board text added: "v1.0 JH 2021 KMŽ Brno I"

Commit message: Add silkscreen place for Vdrop.
Other:
- board text added: "DCC rectifier"
- board text added: "V"
- board text added: "Úbytek napětí:"
- board text removed: "Track voltage rectifier"
